File: MotorDriverPCB/MotorDriverPCB.kicad_sch (KiCad schematic)
At the start: 10 parts

Commit message: Added Encoders
Parts:
- removed MOTOR1, MOTOR2, MOTOR3: Conn_01x02_Pin, Connector_PinHeader_2.54mm:PinHeader_1x02_P2.54mm_Vertical, symbol Connector:Conn_01x02_Pin
- added J1: Conn_02x02_Counter_Clockwise, Connector_PinHeader_2.54mm:PinHeader_2x02_P2.54mm_Vertical, symbol Connector_Generic:Conn_02x02_Counter_Clockwise
- added M1, M2, M3: Conn_02x03_Counter_Clockwise, Headers:Header_02x03, symbol Connector_Generic:Conn_02x03_Counter_Clockwise
Connections:
- net 3V3: now also M1.5 (Pin_5), M2.5 (Pin_5), M3.5 (Pin_5)
- net BAT: now also J1.1 (Pin_1); no longer SW_ARDUINO1.2 (B)
- net BAT_SW: no longer DRIVER1.1 (EN1,2), DRIVER1.16 (VCC1), DRIVER1.9 (EN3,4), DRIVER2.1 (EN1,2), DRIVER2.16 (VCC1)
- net FOR3: now also ESP1.P19 (GPIO19); no longer ESP1.P27 (GPIO27)
- net GND: now also J1.3 (Pin_3), J1.4 (Pin_4), M1.2 (Pin_2), M2.2 (Pin_2), M3.2 (Pin_2)
- net M1F: now also M1.1 (Pin_1)
- net M1R: now also M1.6 (Pin_6)
- net M2F: now also M2.1 (Pin_1)
- net M2R: now also M2.6 (Pin_6)
- net M3F: now also M3.1 (Pin_1)
- net M3R: now also M3.6 (Pin_6)
- net REV3: now also ESP1.P18 (GPIO18); no longer ESP1.P14 (GPIO15)
- net B3: now reaches ESP1.P16 (GPIO16)
- net B3: now also M3.4 (Pin_4)
- net A3: now reaches ESP1.P17 (GPIO17)
- net A3: now also M3.3 (Pin_3)
- net B1: now reaches ESP1.P34 (GPIO34)
- net B1: now also M1.4 (Pin_4)
- net A1: now reaches ESP1.P35 (GPIO35)
- net A1: now also M1.3 (Pin_3)
- new net A2: ESP1.P14 (GPIO15), M2.3 (Pin_3)
- new net B2: ESP1.P27 (GPIO27), M2.4 (Pin_4)
- new net BUCK: DRIVER1.1 (EN1,2), DRIVER1.16 (VCC1), DRIVER1.9 (EN3,4), DRIVER2.1 (EN1,2), DRIVER2.16 (VCC1), J1.2 (Pin_2), SW_ARDUINO1.2 (B)
Other:
- note added: "BuckConverter for ESP"
- note added: "MPU-6050"
- note added: "Motors w/ Encoder"
- note removed: "MOTORS"
- moved on the sheet: BATTERY1, SW_ARDUINO1, SW_BAT1, U1
